Commit message: patched to humble and added bringup and namespace

File: jackal_description/urdf/accessories.urdf.xacro (robot description, xacro)
@@ -4,5 +4,5 @@
     As you add to this URDF, please be aware that both the robot and
     simulation include it. You must retain compatibility with all of
-    the following launch files:
+    the following launch files
     jackal_viz/launch/view_model.launch
     jackal_gazebo/launch/jackal_world.launch
@@ -351,5 +351,5 @@
         <origin xyz="0 0 0" rpy="0 0 0"/>
         <geometry>
-          <mesh filename="package://jackal_description/meshes/ark_enclosure.stl"/>
+          <mesh filename="file://$(find jackal_description)/meshes/ark_enclosure.stl"/>
         </geometry>
         <material name="dark_grey" />

File: jackal_description/urdf/accessories/bridge_plate.urdf.xacro (robot description, xacro)
@@ -17,5 +17,5 @@
         <origin xyz="0 0 0" rpy="1.5707 0.0 1.5707" />
         <geometry>
-          <mesh filename="package://jackal_description/meshes/bridge-plate.stl"/>
+          <mesh filename="file://$(find jackal_description)/meshes/bridge-plate.stl"/>
         </geometry>
         <material name="dark_grey" />

File: jackal_description/urdf/accessories/camera_mount.urdf.xacro (robot description, xacro)
@@ -5,5 +5,5 @@
         <origin xyz="0 0 0" rpy="1.5707 0 1.5707" />
         <geometry>
-          <mesh filename="package://jackal_description/meshes/camera-bracket.stl" scale="0.001 0.001 0.001" />
+          <mesh filename="file://$(find jackal_description)/meshes/camera-bracket.stl" scale="0.001 0.001 0.001" />
         </geometry>
         <material name="dark_grey" />
@@ -14,5 +14,5 @@
         <origin xyz="0 0 0" rpy="0 0 1.5707" />
         <geometry>
-          <mesh filename="package://jackal_description/meshes/camera-beam.stl" scale="0.001 0.001 0.001" />
+          <mesh filename="file://$(find jackal_description)/meshes/camera-beam.stl" scale="0.001 0.001 0.001" />
         </geometry>
         <material name="dark_grey" />

File: jackal_description/urdf/accessories/hdl32_mount.urdf.xacro (robot description, xacro)
@@ -6,5 +6,5 @@
         <visual>
           <geometry>
-            <mesh filename="package://jackal_description/meshes/velodyne_tower.stl"/>
+            <mesh filename="file://$(find jackal_description)/meshes/velodyne_tower.stl"/>
           </geometry>
           <origin xyz="0 0 0" rpy="0 0 0" />
@@ -13,5 +13,5 @@
         <collision>
           <geometry>
-            <mesh filename="package://jackal_description/meshes/velodyne_tower.stl"/>
+            <mesh filename="file://$(find jackal_description)/meshes/velodyne_tower.stl"/>
           </geometry>
           <origin xyz="0 0 0" rpy="0 0 0" />

File: jackal_description/urdf/accessories/hokuyo_ust10.urdf.xacro (robot description, xacro)
@@ -61,5 +61,5 @@
         <geometry>
           <!-- Origin of this mesh is the base of the bracket. -->
-          <mesh filename="package://jackal_description/meshes/hokuyo_ust10.stl" />
+          <mesh filename="file://$(find jackal_description)/meshes/hokuyo_ust10.stl" />
         </geometry>
         <material name="dark_grey" />

File: jackal_description/urdf/accessories/novatel_smart6.urdf.xacro (robot description, xacro)
@@ -6,5 +6,5 @@
       <origin xyz="0 0 0" rpy="0 0 0" />
       <geometry>
-        <mesh filename="package://jackal_description/meshes/novatel-smart6.stl"/>
+        <mesh filename="file://$(find jackal_description)/meshes/novatel-smart6.stl"/>
       </geometry>
       <material name="novatel_white">

File: jackal_description/urdf/accessories/novatel_smart7.urdf.xacro (robot description, xacro)
@@ -6,5 +6,5 @@
         <origin xyz="-0.095 0 0" rpy="${pi/2} 0 -${pi/2}" />
         <geometry>
-          <mesh filename="package://jackal_description/meshes/novatel-smart7.stl"/>
+          <mesh filename="file://$(find jackal_description)/meshes/novatel-smart7.stl"/>
         </geometry>
         <material name="novatel_white">
@@ -15,5 +15,5 @@
         <origin xyz="-0.095 0 0" rpy="${pi/2} 0 -${pi/2}" />
         <geometry>
-          <mesh filename="package://jackal_description/meshes/novatel-smart7.stl"/>
+          <mesh filename="file://$(find jackal_description)/meshes/novatel-smart7.stl"/>
         </geometry>
       </collision>

File: jackal_description/urdf/accessories/sick_lms1xx_mount.urdf.xacro (robot description, xacro)
@@ -39,5 +39,5 @@
         <geometry>
           <!-- Origin of this mesh is the base of the bracket. -->
-          <mesh filename="package://jackal_description/meshes/sick-lms1xx-bracket.stl" />
+          <mesh filename="file://$(find jackal_description)/meshes/sick-lms1xx-bracket.stl" />
         </geometry>
         <material name="dark_grey" />

File: jackal_description/urdf/accessories/stereo_camera_mount.urdf.xacro (robot description, xacro)
@@ -6,5 +6,5 @@
         <origin xyz="0 0 0" rpy="0 0 0" />
         <geometry>
-          <mesh filename="package://jackal_description/meshes/stereo-camera-bracket.stl" />
+          <mesh filename="file://$(find jackal_description)/meshes/stereo-camera-bracket.stl" />
         </geometry>
         <material name="dark_grey" />
@@ -15,5 +15,5 @@
         <origin xyz="0 0 0" rpy="0 0 0" />
         <geometry>
-          <mesh filename="package://jackal_description/meshes/stereo-camera-beam.stl" />
+          <mesh filename="file://$(find jackal_description)/meshes/stereo-camera-beam.stl" />
         </geometry>
         <material name="dark_grey" />

File: jackal_description/urdf/jackal.urdf.xacro (robot description, xacro)
@@ -1,6 +1,7 @@
 <?xml version="1.0"?>
 <robot name="jackal" xmlns:xacro="http://www.ros.org/wiki/xacro">
-  <xacro:arg name="is_sim" default="false" />
-  <xacro:arg name="prefix" default="" />
+  <xacro:arg name="is_sim" default="true" />
+  <xacro:arg name="prefix" default="jackal" />
+  <!-- <xacro:property name="prefix" default="$(arg prefix)" /> -->
   <xacro:arg name="gazebo_controllers" default="$(find jackal_control)/config/control.yaml" />
   <xacro:property name="PI" value="3.1415926535897931" />
@@ -20,10 +21,10 @@
   <material name="yellow"><color rgba="0.8 0.8 0.0 1.0" /></material>
   <material name="black"><color rgba="0.15 0.15 0.15 1.0" /></material>
-  <xacro:macro name="wheel" params="prefix *joint_pose">
-    <link name="${prefix}_wheel_link">
+  <xacro:macro name="wheel" params="wheel_prefix *joint_pose">
+    <link name="${wheel_prefix}_wheel_link">
       <visual>
         <origin xyz="0 0 0" rpy="${PI/2} 0 0"/>
         <geometry>
-          <mesh filename="package://jackal_description/meshes/jackal-wheel.stl"/>
+          <mesh filename="file://$(find jackal_description)/meshes/jackal-wheel.stl"/>
         </geometry>
         <material name="black" />
@@ -44,5 +45,5 @@
       </inertial>
     </link>
-    <gazebo reference="${prefix}_wheel_link">
+    <gazebo reference="${wheel_prefix}_wheel_link">
       <material>Gazebo/DarkGrey</material>
       <selfCollide>false</selfCollide>
@@ -53,7 +54,7 @@
       <fdir1 value="1 0 0"/>
     </gazebo>
-    <joint name="${prefix}_wheel_joint" type="continuous">
-      <parent link="chassis_link"/>
-      <child link="${prefix}_wheel_link" />
+    <joint name="${wheel_prefix}_wheel_joint" type="continuous">
+      <parent link="$(arg prefix)_chassis_link"/>
+      <child link="${wheel_prefix}_wheel_link" />
       <xacro:insert_block name="joint_pose" />
       <axis xyz="0 1 0" />
@@ -61,37 +62,37 @@
     <!-- In reality, Jackal has only two motors, one per side. However, it's more
          straightforward for Gazebo to simulate as if there's an actuator per wheel. -->
-    <transmission name="${prefix}_wheel_trans">
+    <transmission name="${wheel_prefix}_wheel_trans">
       <type>transmission_interface/SimpleTransmission</type>
-      <joint name="${prefix}_wheel">
+      <joint name="${wheel_prefix}_wheel">
         <hardwareInterface>hardware_interface/VelocityJointInterface</hardwareInterface>
       </joint>
-      <actuator name="${prefix}_actuator">
+      <actuator name="${wheel_prefix}_actuator">
         <mechanicalReduction>1</mechanicalReduction>
       </actuator>
     </transmission>
   </xacro:macro>
-  <xacro:wheel prefix="front_left">
+  <xacro:wheel wheel_prefix="$(arg prefix)_front_left">
     <origin xyz="${wheelbase/2} ${track/2} ${wheel_vertical_offset}" rpy="0 0 0" />
   </xacro:wheel>
-  <xacro:wheel prefix="front_right">
+  <xacro:wheel wheel_prefix="$(arg prefix)_front_right">
     <origin xyz="${wheelbase/2} ${-track/2} ${wheel_vertical_offset}" rpy="0 0 0" />
   </xacro:wheel>
-  <xacro:wheel prefix="rear_left">
+  <xacro:wheel wheel_prefix="$(arg prefix)_rear_left">
     <origin xyz="${-wheelbase/2} ${track/2} ${wheel_vertical_offset}" rpy="0 0 0" />
   </xacro:wheel>
-  <xacro:wheel prefix="rear_right">
+  <xacro:wheel wheel_prefix="$(arg prefix)_rear_right">
     <origin xyz="${-wheelbase/2} ${-track/2} ${wheel_vertical_offset}" rpy="0 0 0" />
   </xacro:wheel>
-  <link name="base_link"></link>
-  <joint name="base_link_joint" type="fixed">
+  <link name="$(arg prefix)_base_link"></link>
+  <joint name="$(arg prefix)_base_link_joint" type="fixed">
     <origin xyz="0 0 0" rpy="0 0 0" />
-    <parent link="base_link"/>
-    <child link="chassis_link" />
-  </joint>
-  <link name="chassis_link">
+    <parent link="$(arg prefix)_base_link"/>
+    <child link="$(arg prefix)_chassis_link" />
+  </joint>
+  <link name="$(arg prefix)_chassis_link">
     <visual>
       <origin xyz="0 0 ${footprint_vertical_offset}" rpy="${PI/2} 0 ${PI/2}"/>
       <geometry>
-        <mesh filename="package://jackal_description/meshes/jackal-base.stl"/>
+        <mesh filename="file://$(find jackal_description)/meshes/jackal-base.stl"/>
       </geometry>
       <material name="dark_grey" />
@@ -107,16 +108,15 @@
       <origin xyz="0.012  0.002 0.067" rpy="0 0 0"/>
       <mass value="16.523"/>
-      <!-- Moments of inertia: ( chassis without wheels ) -->
       <inertia
         ixx="0.3136" ixy="-0.0008" ixz="0.0164"
         iyy="0.3922" iyz="-0.0009"
         izz="0.4485"/>
-      </inertial>
+    </inertial>
   </link>
   <xacro:unless value="$(optenv JACKAL_FRONT_ACCESSORY_FENDER 0)">
-    <link name="front_fender_link">
-      <visual>
-        <geometry>
-          <mesh filename="package://jackal_description/meshes/jackal-fender.stl"/>
+    <link name="$(arg prefix)_front_fender_link">
+      <visual>
+        <geometry>
+          <mesh filename="file://$(find jackal_description)/meshes/jackal-fender.stl"/>
         </geometry>
         <material name="yellow" />
@@ -125,29 +125,29 @@
   </xacro:unless>
   <xacro:if value="$(optenv JACKAL_FRONT_ACCESSORY_FENDER 0)">
-    <link name="front_fender_link">
-      <visual>
-        <geometry>
-          <mesh filename="package://jackal_description/meshes/accessory_fender.stl"/>
-        </geometry>
-        <material name="yellow" />
-      </visual>
-    </link>
-    <link name="front_fender_accessory_link"/>
-    <joint name="front_fender_accessory_joint" type="fixed">
+    <link name="$(arg prefix)_front_fender_link">
+      <visual>
+        <geometry>
+          <mesh filename="file://$(find jackal_description)/meshes/accessory_fender.stl"/>
+        </geometry>
+        <material name="yellow" />
+      </visual>
+    </link>
+    <link name="$(arg prefix)_front_fender_accessory_link"/>
+    <joint name="$(arg prefix)_front_fender_accessory_joint" type="fixed">
       <origin xyz="0.25629 0 0.07455" rpy="${PI} 0 0" />
-      <parent link="front_fender_link" />
-      <child link="front_fender_accessory_link" />
+      <parent link="$(arg prefix)_front_fender_link" />
+      <child link="$(arg prefix)_front_fender_accessory_link" />
     </joint>
   </xacro:if>
-  <joint name="front_fender_joint" type="fixed">
+  <joint name="$(arg prefix)_front_fender_joint" type="fixed">
     <origin xyz="0 0 0" rpy="0 0 0"/>
-    <parent link="chassis_link" />
-    <child link="front_fender_link" />
+    <parent link="$(arg prefix)_chassis_link" />
+    <child link="$(arg prefix)_front_fender_link" />
   </joint>
   <xacro:unless value="$(optenv JACKAL_REAR_ACCESSORY_FENDER 0)">
-    <link name="rear_fender_link">
-      <visual>
-        <geometry>
-          <mesh filename="package://jackal_description/meshes/jackal-fender.stl"/>
+    <link name="$(arg prefix)_rear_fender_link">
+      <visual>
+        <geometry>
+          <mesh filename="file://$(find jackal_description)/meshes/jackal-fender.stl"/>
         </geometry>
         <material name="yellow" />
@@ -156,29 +156,29 @@
   </xacro:unless>
   <xacro:if value="$(optenv JACKAL_REAR_ACCESSORY_FENDER 0)">
-    <link name="rear_fender_link">
-      <visual>
-        <geometry>
-          <mesh filename="package://jackal_description/meshes/accessory_fender.stl"/>
-        </geometry>
-        <material name="yellow" />
-      </visual>
-    </link>
-    <link name="rear_fender_accessory_link"/>
-    <joint name="rear_fender_accessory_joint" type="fixed">
+    <link name="$(arg prefix)_rear_fender_link">
+      <visual>
+        <geometry>
+          <mesh filename="file://$(find jackal_description)/meshes/accessory_fender.stl"/>
+        </geometry>
+        <material name="yellow" />
+      </visual>
+    </link>
+    <link name="$(arg prefix)_rear_fender_accessory_link"/>
+    <joint name="$(arg prefix)_rear_fender_accessory_joint" type="fixed">
       <origin xyz="0.25629 0 0.07455" rpy="${PI} 0 0" />
-      <parent link="rear_fender_link" />
-      <child link="rear_fender_accessory_link" />
+      <parent link="$(arg prefix)_rear_fender_link" />
+      <child link="$(arg prefix)_rear_fender_accessory_link" />
     </joint>
   </xacro:if>
-  <joint name="rear_fender_joint" type="fixed">
+  <joint name="$(arg prefix)_rear_fender_joint" type="fixed">
     <origin xyz="0 0 0" rpy="0 0 ${PI}"/>
-    <parent link="chassis_link" />
-    <child link="rear_fender_link" />
-  </joint>
-  <!-- TODO: Make this internal_imu_link or something, and use a mixed-in xacro
+    <parent link="$(arg prefix)_chassis_link" />
+    <child link="$(arg prefix)_rear_fender_link" />
+  </joint>
+  <!-- TODO Make this internal_imu_link or something, and use a mixed-in xacro
        to supply the joint between it and imu_link. This is important so that imu_link
        always points to the "active" IMU. When an upgrade IMU is connected, the
        internal_imu_link should remain, but imu_link should point to the upgrade one. -->
-  <link name="imu_link">
+  <link name="$(arg prefix)_imu_link">
     <inertial>
       <mass value="0.001"/>
@@ -187,10 +187,10 @@
     </inertial>
   </link>
-  <joint name="imu_joint" type="fixed">
-    <parent link="chassis_link" />
-    <child link="imu_link" />
-  </joint>
-  <!-- TODO: Same note as applies to imu_link -->
-  <link name="navsat_link">
+  <joint name="$(arg prefix)_imu_joint" type="fixed">
+    <parent link="$(arg prefix)_chassis_link" />
+    <child link="$(arg prefix)_imu_link" />
+  </joint>
+  <!-- TODO Same note as applies to imu_link -->
+  <link name="$(arg prefix)_navsat_link">
     <visual>
       <geometry>
@@ -201,25 +201,25 @@
     </visual>
   </link>
-  <joint name="navsat_joint" type="fixed">
-    <parent link="chassis_link" />
-    <child link="navsat_link" />
+  <joint name="$(arg prefix)_navsat_joint" type="fixed">
+    <parent link="$(arg prefix)_chassis_link" />
+    <child link="$(arg prefix)_navsat_link" />
     <origin xyz="-0.180 0.126 0.1815" />
   </joint>
-  <link name="mid_mount"></link>
-  <joint name="mid_mount_joint" type="fixed">
-    <parent link="chassis_link" />
-    <child link="mid_mount" />
+  <link name="$(arg prefix)_mid_mount"></link>
+  <joint name="$(arg prefix)_mid_mount_joint" type="fixed">
+    <parent link="$(arg prefix)_chassis_link" />
+    <child link="$(arg prefix)_mid_mount" />
     <origin xyz="0 0 ${chassis_height}" />
   </joint>
-  <link name="rear_mount"></link>
-  <joint name="rear_mount_joint" type="fixed">
-    <parent link="mid_mount" />
-    <child link="rear_mount" />
+  <link name="$(arg prefix)_rear_mount"></link>
+  <joint name="$(arg prefix)_rear_mount_joint" type="fixed">
+    <parent link="$(arg prefix)_mid_mount" />
+    <child link="$(arg prefix)_rear_mount" />
     <origin xyz="${-mount_spacing} 0 0" />
   </joint>
-  <link name="front_mount"></link>
-  <joint name="front_mount_joint" type="fixed">
-    <parent link="mid_mount" />
-    <child link="front_mount" />
+  <link name="$(arg prefix)_front_mount"></link>
+  <joint name="$(arg prefix)_front_mount_joint" type="fixed">
+    <parent link="$(arg prefix)_mid_mount" />
+    <child link="$(arg prefix)_front_mount" />
     <origin xyz="${mount_spacing} 0 0" />
   </joint>
@@ -235,20 +235,20 @@
       </xacro:unless>
     </hardware>
-    <joint name="front_left_wheel_joint">
-      <command_interface name="velocity"/>
-      <state_interface name="position"/>
-      <state_interface name="velocity"/>
-    </joint>
-    <joint name="rear_left_wheel_joint">
-      <command_interface name="velocity"/>
-      <state_interface name="position"/>
-      <state_interface name="velocity"/>
-    </joint>
-    <joint name="front_right_wheel_joint">
-      <command_interface name="velocity"/>
-      <state_interface name="position"/>
-      <state_interface name="velocity"/>
-    </joint>
-    <joint name="rear_right_wheel_joint">
+    <joint name="$(arg prefix)_front_left_wheel_joint">
+      <command_interface name="velocity"/>
+      <state_interface name="position"/>
+      <state_interface name="velocity"/>
+    </joint>
+    <joint name="$(arg prefix)_rear_left_wheel_joint">
+      <command_interface name="velocity"/>
+      <state_interface name="position"/>
+      <state_interface name="velocity"/>
+    </joint>
+    <joint name="$(arg prefix)_front_right_wheel_joint">
+      <command_interface name="velocity"/>
+      <state_interface name="position"/>
+      <state_interface name="velocity"/>
+    </joint>
+    <joint name="$(arg prefix)_rear_right_wheel_joint">
       <command_interface name="velocity"/>
       <state_interface name="position"/>
@@ -257,7 +257,7 @@
   </ros2_control>
   <!-- Bring in simulation data for Gazebo. -->
-  <xacro:if value="$(arg is_sim)">
-    <xacro:include filename="$(find jackal_description)/urdf/jackal.gazebo" />
-  </xacro:if>
+  <!-- <xacro:if value="$(arg is_sim)"> -->
+  <xacro:include filename="$(find jackal_description)/urdf/jackal.gazebo" />
+  <!-- </xacro:if> -->
   <!-- Optional standard accessories, including their simulation data. The rendering
        of these into the final description is controlled by optenv variables, which
