Commit message: fix: jackal colors

File: jackal_description/urdf/accessories.urdf.xacro (robot description, xacro)
@@ -14,9 +14,9 @@
   <xacro:include filename="$(find jackal_description)/urdf/accessories/bridge_plate.urdf.xacro" />
   <!-- 2D Lidars -->
-  <!-- <xacro:include filename="$(find lms1xx)/urdf/sick_lms1xx.urdf.xacro" />
-  <xacro:include filename="$(find jackal_description)/urdf/accessories/sick_lms1xx_mount.urdf.xacro" />-->
+  <!-- <xacro:include filename="$(find lms1xx)/urdf/sick_lms1xx.urdf.xacro" />  -->
+  <!-- <xacro:include filename="$(find jackal_description)/urdf/accessories/sick_lms1xx_mount.urdf.xacro" /> -->
   <xacro:include filename="$(find jackal_description)/urdf/accessories/hokuyo_ust10.urdf.xacro" />
-  <xacro:include filename="$(find jackal_description)/urdf/accessories/vlp16_mount.urdf.xacro" />
-  <xacro:include filename="$(find jackal_description)/urdf/accessories/hdl32_mount.urdf.xacro" />
+  <!-- <xacro:include filename="$(find jackal_description)/urdf/accessories/vlp16_mount.urdf.xacro" />
+  <xacro:include filename="$(find jackal_description)/urdf/accessories/hdl32_mount.urdf.xacro" /> -->
   <!--
     Add primary/secondary 2D lidar sensors.  By default these are SICK LMS1xx but can be changed with the
@@ -26,14 +26,15 @@
   -->
   <!-- Primary 2D Lidar -->
-  <xacro:if value="$(optenv JACKAL_LASER 0)">
+  <xacro:property name="laser" value="$(optenv JACKAL_LASER 1)" />
+  <xacro:if value="${laser}">
     <xacro:property name="mount" value="$(optenv JACKAL_LASER_MOUNT front)" />
-    <xacro:property name="topic" value="$(optenv JACKAL_LASER_TOPIC front/scan)" />
-    <xacro:property name="tower" value="$(optenv JACKAL_LASER_TOWER 1)" />
+    <xacro:property name="topic" value="$(optenv JACKAL_LASER_TOPIC scan)" />
+    <xacro:property name="tower" value="$(optenv JACKAL_LASER_TOWER 0)" />
     <xacro:property name="prefix" value="$(optenv JACKAL_LASER_PREFIX ${mount})" />
-    <xacro:property name="parent" value="$(optenv JACKAL_LASER_PARENT ${mount}_mount)" />
+    <xacro:property name="parent" value="$(optenv JACKAL_LASER_PARENT jackal/${mount}_mount)" />
     <xacro:property name="lidar_model" value="$(optenv JACKAL_LASER_MODEL ust10)" />
     <!-- SICK LMS1xx -->
-    <xacro:if value="${lidar_model == 'lms1xx'}">
-      <!-- Mount Enabled -->
+    <!-- <xacro:if value="${lidar_model == 'lms1xx'}">
+       Mount Enabled
       <xacro:if value="${tower}">
         <xacro:sick_lms1xx_mount topic="${topic}" prefix="${prefix}" parent_link="${parent}">
@@ -41,5 +42,5 @@
         </xacro:sick_lms1xx_mount>
       </xacro:if>
-      <!-- Mount Disabled -->
+       Mount Disabled
       <xacro:unless value="${tower}">
         <xacro:sick_lms1xx frame="${prefix}_laser" topic="${topic}" />
@@ -56,8 +57,8 @@
         </joint>
       </xacro:unless>
-    </xacro:if>
+    </xacro:if> -->
     <!-- Hokuyo UST10 -->
     <xacro:if value="${lidar_model == 'ust10'}">
-      <xacro:hokuyo_ust10_mount topic="${topic}" prefix="${prefix}" parent_link="${parent}">
+      <xacro:hokuyo_ust10_mount topic="${topic}" prefix="jackal/front" parent_link="${parent}">
         <origin xyz="$(optenv JACKAL_LASER_OFFSET 0 0 0)" rpy="$(optenv JACKAL_LASER_RPY 0 0 0)" />
       </xacro:hokuyo_ust10_mount>
@@ -65,5 +66,5 @@
   </xacro:if>
   <!-- Secondary 2D Lidar -->
-  <xacro:if value="$(optenv JACKAL_LASER_SECONDARY 0)">
+  <!-- <xacro:if value="$(optenv JACKAL_LASER_SECONDARY 0)">
     <xacro:property name="mount" value="$(optenv JACKAL_LASER_SECONDARY_MOUNT rear)" />
     <xacro:property name="topic" value="$(optenv JACKAL_LASER_SECONDARY_TOPIC rear/scan)" />
@@ -72,7 +73,5 @@
     <xacro:property name="parent" value="$(optenv JACKAL_LASER_SECONDARY_PARENT ${mount}_mount)" />
     <xacro:property name="lidar_model" value="$(optenv JACKAL_LASER_SECONDARY_MODEL ust10)" />
-    <!-- SICK LMS1xx -->
     <xacro:if value="${lidar_model == 'lms1xx'}">
-      <!-- Mount Enabled -->
       <xacro:if value="${tower}">
         <xacro:sick_lms1xx_mount topic="${topic}" prefix="${prefix}" parent_link="${parent}">
@@ -80,5 +79,4 @@
         </xacro:sick_lms1xx_mount>
       </xacro:if>
-      <!-- Mount Disabled -->
       <xacro:unless value="${tower}">
         <xacro:sick_lms1xx frame="${prefix}_laser" topic="${topic}" />
@@ -96,5 +94,4 @@
       </xacro:unless>
     </xacro:if>
-    <!-- Hokuyo UST10 -->
     <xacro:if value="${lidar_model == 'ust10'}">
       <xacro:hokuyo_ust10_mount topic="${topic}" prefix="${prefix}" parent_link="${parent}">
@@ -102,5 +99,5 @@
       </xacro:hokuyo_ust10_mount>
     </xacro:if>
-  </xacro:if>
+  </xacro:if> -->
   <!--
     Add a 3D lidar sensor.  By default this is a Velodyne VLP16 but can be changed with the

File: jackal_description/urdf/accessories/hokuyo_ust10.urdf.xacro (robot description, xacro)
@@ -41,9 +41,15 @@
           <plugin name="gazebo_ros_laser" filename="libgazebo_ros_ray_sensor.so">
             <ros>
+              <qos>
+                <publisher>
+                  <reliability>best_effort</reliability>
+                  <durability>volatile</durability>
+                </publisher>
+              </qos>
               <namespace>${robot_namespace}</namespace>
               <remapping>~/out:=${topic}</remapping>
             </ros>
             <output_type>sensor_msgs/LaserScan</output_type>
-            <frame_name>${frame}</frame_name>
+            <frame_name>jackal/front_laser</frame_name>
           </plugin>
         </sensor>

File: jackal_description/urdf/accessories/sick_lms1xx_mount.urdf.xacro (robot description, xacro)
@@ -26,5 +26,5 @@
 -->
 <robot xmlns:xacro="http://www.ros.org/wiki/xacro">
-  <xacro:include filename="$(find lms1xx)/urdf/sick_lms1xx.urdf.xacro" />
+  <!-- <xacro:include filename="$(find lms1xx)/urdf/sick_lms1xx.urdf.xacro" /> -->
   <xacro:macro name="sick_lms1xx_mount" params="prefix topic parent_link *origin">
     <xacro:sick_lms1xx frame="${prefix}_laser" topic="${topic}" />

File: jackal_description/urdf/jackal.urdf.xacro (robot description, xacro)
@@ -33,5 +33,5 @@
         <origin xyz="0 0 0" rpy="${PI/2} 0 0"/>
         <geometry>
-          <cylinder radius="${wheel_radius}" length="${wheel_width}"/>
+          <sphere radius="${wheel_radius}"/>
         </geometry>
       </collision>
@@ -48,6 +48,6 @@
       <material>Gazebo/DarkGrey</material>
       <selfCollide>false</selfCollide>
-      <mu1 value="0.5"/>
-      <mu2 value="0.5"/>
+      <mu1 value="3.5"/>
+      <mu2 value="10.2"/>
       <kp value="10000000.0" />
       <kd value="1" />
@@ -55,5 +55,5 @@
     </gazebo>
     <joint name="${wheel_prefix}_wheel_joint" type="continuous">
-      <parent link="$(arg prefix)_chassis_link"/>
+      <parent link="$(arg prefix)/chassis_link"/>
       <child link="${wheel_prefix}_wheel_link" />
       <xacro:insert_block name="joint_pose" />
@@ -72,23 +72,23 @@
     </transmission>
   </xacro:macro>
-  <xacro:wheel wheel_prefix="$(arg prefix)_front_left">
+  <xacro:wheel wheel_prefix="$(arg prefix)/front_left">
     <origin xyz="${wheelbase/2} ${track/2} ${wheel_vertical_offset}" rpy="0 0 0" />
   </xacro:wheel>
-  <xacro:wheel wheel_prefix="$(arg prefix)_front_right">
+  <xacro:wheel wheel_prefix="$(arg prefix)/front_right">
     <origin xyz="${wheelbase/2} ${-track/2} ${wheel_vertical_offset}" rpy="0 0 0" />
   </xacro:wheel>
-  <xacro:wheel wheel_prefix="$(arg prefix)_rear_left">
+  <xacro:wheel wheel_prefix="$(arg prefix)/rear_left">
     <origin xyz="${-wheelbase/2} ${track/2} ${wheel_vertical_offset}" rpy="0 0 0" />
   </xacro:wheel>
-  <xacro:wheel wheel_prefix="$(arg prefix)_rear_right">
+  <xacro:wheel wheel_prefix="$(arg prefix)/rear_right">
     <origin xyz="${-wheelbase/2} ${-track/2} ${wheel_vertical_offset}" rpy="0 0 0" />
   </xacro:wheel>
-  <link name="$(arg prefix)_base_link"></link>
-  <joint name="$(arg prefix)_base_link_joint" type="fixed">
+  <link name="$(arg prefix)/base_link"></link>
+  <joint name="$(arg prefix)/base_link_joint" type="fixed">
     <origin xyz="0 0 0" rpy="0 0 0" />
-    <parent link="$(arg prefix)_base_link"/>
-    <child link="$(arg prefix)_chassis_link" />
-  </joint>
-  <link name="$(arg prefix)_chassis_link">
+    <parent link="$(arg prefix)/base_link"/>
+    <child link="$(arg prefix)/chassis_link" />
+  </joint>
+  <link name="$(arg prefix)/chassis_link">
     <visual>
       <origin xyz="0 0 ${footprint_vertical_offset}" rpy="${PI/2} 0 ${PI/2}"/>
@@ -114,6 +114,9 @@
     </inertial>
   </link>
+  <!-- <gazebo reference="$(arg prefix)/chassis_link">
+      <material>Gazebo/DarkGrey</material>
+    </gazebo> -->
   <xacro:unless value="$(optenv JACKAL_FRONT_ACCESSORY_FENDER 0)">
-    <link name="$(arg prefix)_front_fender_link">
+    <link name="$(arg prefix)/front_fender_link">
       <visual>
         <geometry>
@@ -123,7 +126,10 @@
       </visual>
     </link>
+    <!-- <gazebo reference="$(arg prefix)/front_fender_link">
+      <material>Gazebo/Yellow</material>
+    </gazebo> -->
   </xacro:unless>
   <xacro:if value="$(optenv JACKAL_FRONT_ACCESSORY_FENDER 0)">
-    <link name="$(arg prefix)_front_fender_link">
+    <link name="$(arg prefix)/front_fender_link">
       <visual>
         <geometry>
@@ -133,18 +139,21 @@
       </visual>
     </link>
-    <link name="$(arg prefix)_front_fender_accessory_link"/>
-    <joint name="$(arg prefix)_front_fender_accessory_joint" type="fixed">
+    <!-- <gazebo reference="$(arg prefix)/front_fender_link">
+      <material>Gazebo/Yellow</material>
+    </gazebo> -->
+    <link name="$(arg prefix)/front_fender_accessory_link"/>
+    <joint name="$(arg prefix)/front_fender_accessory_joint" type="fixed">
       <origin xyz="0.25629 0 0.07455" rpy="${PI} 0 0" />
-      <parent link="$(arg prefix)_front_fender_link" />
-      <child link="$(arg prefix)_front_fender_accessory_link" />
+      <parent link="$(arg prefix)/front_fender_link" />
+      <child link="$(arg prefix)/front_fender_accessory_link" />
     </joint>
   </xacro:if>
-  <joint name="$(arg prefix)_front_fender_joint" type="fixed">
+  <joint name="$(arg prefix)/front_fender_joint" type="fixed">
     <origin xyz="0 0 0" rpy="0 0 0"/>
-    <parent link="$(arg prefix)_chassis_link" />
-    <child link="$(arg prefix)_front_fender_link" />
+    <parent link="$(arg prefix)/chassis_link" />
+    <child link="$(arg prefix)/front_fender_link" />
   </joint>
   <xacro:unless value="$(optenv JACKAL_REAR_ACCESSORY_FENDER 0)">
-    <link name="$(arg prefix)_rear_fender_link">
+    <link name="$(arg prefix)/rear_fender_link">
       <visual>
         <geometry>
@@ -154,7 +163,10 @@
       </visual>
     </link>
+    <!-- <gazebo reference="$(arg prefix)/rear_fender_link">
+      <material>Gazebo/Yellow</material>
+    </gazebo> -->
   </xacro:unless>
   <xacro:if value="$(optenv JACKAL_REAR_ACCESSORY_FENDER 0)">
-    <link name="$(arg prefix)_rear_fender_link">
+    <link name="$(arg prefix)/rear_fender_link">
       <visual>
         <geometry>
@@ -164,15 +176,18 @@
       </visual>
     </link>
-    <link name="$(arg prefix)_rear_fender_accessory_link"/>
-    <joint name="$(arg prefix)_rear_fender_accessory_joint" type="fixed">
+    <!-- <gazebo reference="$(arg prefix)/rear_fender_link">
+      <material>Gazebo/Yellow</material>
+    </gazebo> -->
+    <link name="$(arg prefix)/rear_fender_accessory_link"/>
+    <joint name="$(arg prefix)/rear_fender_accessory_joint" type="fixed">
       <origin xyz="0.25629 0 0.07455" rpy="${PI} 0 0" />
-      <parent link="$(arg prefix)_rear_fender_link" />
-      <child link="$(arg prefix)_rear_fender_accessory_link" />
+      <parent link="$(arg prefix)/rear_fender_link" />
+      <child link="$(arg prefix)/rear_fender_accessory_link" />
     </joint>
   </xacro:if>
-  <joint name="$(arg prefix)_rear_fender_joint" type="fixed">
+  <joint name="$(arg prefix)/rear_fender_joint" type="fixed">
     <origin xyz="0 0 0" rpy="0 0 ${PI}"/>
-    <parent link="$(arg prefix)_chassis_link" />
-    <child link="$(arg prefix)_rear_fender_link" />
+    <parent link="$(arg prefix)/chassis_link" />
+    <child link="$(arg prefix)/rear_fender_link" />
   </joint>
   <!-- TODO Make this internal_imu_link or something, and use a mixed-in xacro
@@ -180,5 +195,5 @@
        always points to the "active" IMU. When an upgrade IMU is connected, the
        internal_imu_link should remain, but imu_link should point to the upgrade one. -->
-  <link name="$(arg prefix)_imu_link">
+  <link name="$(arg prefix)/imu_link">
     <inertial>
       <mass value="0.001"/>
@@ -187,10 +202,10 @@
     </inertial>
   </link>
-  <joint name="$(arg prefix)_imu_joint" type="fixed">
-    <parent link="$(arg prefix)_chassis_link" />
-    <child link="$(arg prefix)_imu_link" />
+  <joint name="$(arg prefix)/imu_joint" type="fixed">
+    <parent link="$(arg prefix)/chassis_link" />
+    <child link="$(arg prefix)/imu_link" />
   </joint>
   <!-- TODO Same note as applies to imu_link -->
-  <link name="$(arg prefix)_navsat_link">
+  <link name="$(arg prefix)/navsat_link">
     <visual>
       <geometry>
@@ -201,26 +216,29 @@
     </visual>
   </link>
-  <joint name="$(arg prefix)_navsat_joint" type="fixed">
-    <parent link="$(arg prefix)_chassis_link" />
-    <child link="$(arg prefix)_navsat_link" />
+  <!-- <gazebo reference="$(arg prefix)/navsat_link">
+      <material>Gazebo/DarkGrey</material>
+    </gazebo> -->
+  <joint name="$(arg prefix)/navsat_joint" type="fixed">
+    <parent link="$(arg prefix)/chassis_link" />
+    <child link="$(arg prefix)/navsat_link" />
     <origin xyz="-0.180 0.126 0.1815" />
   </joint>
-  <link name="$(arg prefix)_mid_mount"></link>
-  <joint name="$(arg prefix)_mid_mount_joint" type="fixed">
-    <parent link="$(arg prefix)_chassis_link" />
-    <child link="$(arg prefix)_mid_mount" />
+  <link name="$(arg prefix)/mid_mount"></link>
+  <joint name="$(arg prefix)/mid_mount_joint" type="fixed">
+    <parent link="$(arg prefix)/chassis_link" />
+    <child link="$(arg prefix)/mid_mount" />
     <origin xyz="0 0 ${chassis_height}" />
   </joint>
-  <link name="$(arg prefix)_rear_mount"></link>
-  <joint name="$(arg prefix)_rear_mount_joint" type="fixed">
-    <parent link="$(arg prefix)_mid_mount" />
-    <child link="$(arg prefix)_rear_mount" />
+  <link name="$(arg prefix)/rear_mount"></link>
+  <joint name="$(arg prefix)/rear_mount_joint" type="fixed">
+    <parent link="$(arg prefix)/mid_mount" />
+    <child link="$(arg prefix)/rear_mount" />
     <origin xyz="${-mount_spacing} 0 0" />
   </joint>
-  <link name="$(arg prefix)_front_mount"></link>
-  <joint name="$(arg prefix)_front_mount_joint" type="fixed">
-    <parent link="$(arg prefix)_mid_mount" />
-    <child link="$(arg prefix)_front_mount" />
-    <origin xyz="${mount_spacing} 0 0" />
+  <link name="$(arg prefix)/front_mount"></link>
+  <joint name="$(arg prefix)/front_mount_joint" type="fixed">
+    <parent link="$(arg prefix)/mid_mount" />
+    <child link="$(arg prefix)/front_mount" />
+    <origin xyz="0 0 0" />
   </joint>
   <!-- ROS2 controls -->
@@ -235,20 +253,20 @@
       </xacro:unless>
     </hardware>
-    <joint name="$(arg prefix)_front_left_wheel_joint">
-      <command_interface name="velocity"/>
-      <state_interface name="position"/>
-      <state_interface name="velocity"/>
-    </joint>
-    <joint name="$(arg prefix)_rear_left_wheel_joint">
-      <command_interface name="velocity"/>
-      <state_interface name="position"/>
-      <state_interface name="velocity"/>
-    </joint>
-    <joint name="$(arg prefix)_front_right_wheel_joint">
-      <command_interface name="velocity"/>
-      <state_interface name="position"/>
-      <state_interface name="velocity"/>
-    </joint>
-    <joint name="$(arg prefix)_rear_right_wheel_joint">
+    <joint name="$(arg prefix)/front_left_wheel_joint">
+      <command_interface name="velocity"/>
+      <state_interface name="position"/>
+      <state_interface name="velocity"/>
+    </joint>
+    <joint name="$(arg prefix)/rear_left_wheel_joint">
+      <command_interface name="velocity"/>
+      <state_interface name="position"/>
+      <state_interface name="velocity"/>
+    </joint>
+    <joint name="$(arg prefix)/front_right_wheel_joint">
+      <command_interface name="velocity"/>
+      <state_interface name="position"/>
+      <state_interface name="velocity"/>
+    </joint>
+    <joint name="$(arg prefix)/rear_right_wheel_joint">
       <command_interface name="velocity"/>
       <state_interface name="position"/>
