Commit message: fix: urdf fixed, now works on new gazebo

File: jackal_description/urdf/accessories.urdf.xacro (robot description, xacro)
@@ -32,5 +32,5 @@
     <xacro:property name="tower" value="$(optenv JACKAL_LASER_TOWER 0)" />
     <xacro:property name="prefix" value="$(optenv JACKAL_LASER_PREFIX ${mount})" />
-    <xacro:property name="parent" value="$(optenv JACKAL_LASER_PARENT jackal/${mount}_mount)" />
+    <xacro:property name="parent" value="$(optenv JACKAL_LASER_PARENT jackal_${mount}_mount)" />
     <xacro:property name="lidar_model" value="$(optenv JACKAL_LASER_MODEL ust10)" />
     <!-- SICK LMS1xx -->
@@ -60,5 +60,5 @@
     <!-- Hokuyo UST10 -->
     <xacro:if value="${lidar_model == 'ust10'}">
-      <xacro:hokuyo_ust10_mount topic="${topic}" prefix="jackal/front" parent_link="${parent}">
+      <xacro:hokuyo_ust10_mount topic="${topic}" prefix="jackal_front" parent_link="${parent}">
         <origin xyz="$(optenv JACKAL_LASER_OFFSET 0 0 0)" rpy="$(optenv JACKAL_LASER_RPY 0 0 0)" />
       </xacro:hokuyo_ust10_mount>

File: jackal_description/urdf/jackal.urdf.xacro (robot description, xacro)
@@ -55,5 +55,5 @@
     </gazebo>
     <joint name="${wheel_prefix}_wheel_joint" type="continuous">
-      <parent link="$(arg prefix)/chassis_link"/>
+      <parent link="$(arg prefix)_chassis_link"/>
       <child link="${wheel_prefix}_wheel_link" />
       <xacro:insert_block name="joint_pose" />
@@ -72,23 +72,23 @@
     </transmission>
   </xacro:macro>
-  <xacro:wheel wheel_prefix="$(arg prefix)/front_left">
+  <xacro:wheel wheel_prefix="$(arg prefix)_front_left">
     <origin xyz="${wheelbase/2} ${track/2} ${wheel_vertical_offset}" rpy="0 0 0" />
   </xacro:wheel>
-  <xacro:wheel wheel_prefix="$(arg prefix)/front_right">
+  <xacro:wheel wheel_prefix="$(arg prefix)_front_right">
     <origin xyz="${wheelbase/2} ${-track/2} ${wheel_vertical_offset}" rpy="0 0 0" />
   </xacro:wheel>
-  <xacro:wheel wheel_prefix="$(arg prefix)/rear_left">
+  <xacro:wheel wheel_prefix="$(arg prefix)_rear_left">
     <origin xyz="${-wheelbase/2} ${track/2} ${wheel_vertical_offset}" rpy="0 0 0" />
   </xacro:wheel>
-  <xacro:wheel wheel_prefix="$(arg prefix)/rear_right">
+  <xacro:wheel wheel_prefix="$(arg prefix)_rear_right">
     <origin xyz="${-wheelbase/2} ${-track/2} ${wheel_vertical_offset}" rpy="0 0 0" />
   </xacro:wheel>
-  <link name="$(arg prefix)/base_link"></link>
-  <joint name="$(arg prefix)/base_link_joint" type="fixed">
+  <link name="$(arg prefix)_base_link"></link>
+  <joint name="$(arg prefix)_base_link_joint" type="fixed">
     <origin xyz="0 0 0" rpy="0 0 0" />
-    <parent link="$(arg prefix)/base_link"/>
-    <child link="$(arg prefix)/chassis_link" />
-  </joint>
-  <link name="$(arg prefix)/chassis_link">
+    <parent link="$(arg prefix)_base_link"/>
+    <child link="$(arg prefix)_chassis_link" />
+  </joint>
+  <link name="$(arg prefix)_chassis_link">
     <visual>
       <origin xyz="0 0 ${footprint_vertical_offset}" rpy="${PI/2} 0 ${PI/2}"/>
@@ -118,5 +118,5 @@
     </gazebo> -->
   <xacro:unless value="$(optenv JACKAL_FRONT_ACCESSORY_FENDER 0)">
-    <link name="$(arg prefix)/front_fender_link">
+    <link name="$(arg prefix)_front_fender_link">
       <visual>
         <geometry>
@@ -131,5 +131,5 @@
   </xacro:unless>
   <xacro:if value="$(optenv JACKAL_FRONT_ACCESSORY_FENDER 0)">
-    <link name="$(arg prefix)/front_fender_link">
+    <link name="$(arg prefix)_front_fender_link">
       <visual>
         <geometry>
@@ -142,18 +142,18 @@
       <material>Gazebo/Yellow</material>
     </gazebo> -->
-    <link name="$(arg prefix)/front_fender_accessory_link"/>
-    <joint name="$(arg prefix)/front_fender_accessory_joint" type="fixed">
+    <link name="$(arg prefix)_front_fender_accessory_link"/>
+    <joint name="$(arg prefix)_front_fender_accessory_joint" type="fixed">
       <origin xyz="0.25629 0 0.07455" rpy="${PI} 0 0" />
-      <parent link="$(arg prefix)/front_fender_link" />
-      <child link="$(arg prefix)/front_fender_accessory_link" />
+      <parent link="$(arg prefix)_front_fender_link" />
+      <child link="$(arg prefix)_front_fender_accessory_link" />
     </joint>
   </xacro:if>
-  <joint name="$(arg prefix)/front_fender_joint" type="fixed">
+  <joint name="$(arg prefix)_front_fender_joint" type="fixed">
     <origin xyz="0 0 0" rpy="0 0 0"/>
-    <parent link="$(arg prefix)/chassis_link" />
-    <child link="$(arg prefix)/front_fender_link" />
+    <parent link="$(arg prefix)_chassis_link" />
+    <child link="$(arg prefix)_front_fender_link" />
   </joint>
   <xacro:unless value="$(optenv JACKAL_REAR_ACCESSORY_FENDER 0)">
-    <link name="$(arg prefix)/rear_fender_link">
+    <link name="$(arg prefix)_rear_fender_link">
       <visual>
         <geometry>
@@ -168,5 +168,5 @@
   </xacro:unless>
   <xacro:if value="$(optenv JACKAL_REAR_ACCESSORY_FENDER 0)">
-    <link name="$(arg prefix)/rear_fender_link">
+    <link name="$(arg prefix)_rear_fender_link">
       <visual>
         <geometry>
@@ -179,15 +179,15 @@
       <material>Gazebo/Yellow</material>
     </gazebo> -->
-    <link name="$(arg prefix)/rear_fender_accessory_link"/>
-    <joint name="$(arg prefix)/rear_fender_accessory_joint" type="fixed">
+    <link name="$(arg prefix)_rear_fender_accessory_link"/>
+    <joint name="$(arg prefix)_rear_fender_accessory_joint" type="fixed">
       <origin xyz="0.25629 0 0.07455" rpy="${PI} 0 0" />
-      <parent link="$(arg prefix)/rear_fender_link" />
-      <child link="$(arg prefix)/rear_fender_accessory_link" />
+      <parent link="$(arg prefix)_rear_fender_link" />
+      <child link="$(arg prefix)_rear_fender_accessory_link" />
     </joint>
   </xacro:if>
-  <joint name="$(arg prefix)/rear_fender_joint" type="fixed">
+  <joint name="$(arg prefix)_rear_fender_joint" type="fixed">
     <origin xyz="0 0 0" rpy="0 0 ${PI}"/>
-    <parent link="$(arg prefix)/chassis_link" />
-    <child link="$(arg prefix)/rear_fender_link" />
+    <parent link="$(arg prefix)_chassis_link" />
+    <child link="$(arg prefix)_rear_fender_link" />
   </joint>
   <!-- TODO Make this internal_imu_link or something, and use a mixed-in xacro
@@ -195,5 +195,5 @@
        always points to the "active" IMU. When an upgrade IMU is connected, the
        internal_imu_link should remain, but imu_link should point to the upgrade one. -->
-  <link name="$(arg prefix)/imu_link">
+  <link name="$(arg prefix)_imu_link">
     <inertial>
       <mass value="0.001"/>
@@ -202,10 +202,10 @@
     </inertial>
   </link>
-  <joint name="$(arg prefix)/imu_joint" type="fixed">
-    <parent link="$(arg prefix)/chassis_link" />
-    <child link="$(arg prefix)/imu_link" />
+  <joint name="$(arg prefix)_imu_joint" type="fixed">
+    <parent link="$(arg prefix)_chassis_link" />
+    <child link="$(arg prefix)_imu_link" />
   </joint>
   <!-- TODO Same note as applies to imu_link -->
-  <link name="$(arg prefix)/navsat_link">
+  <link name="$(arg prefix)_navsat_link">
     <visual>
       <geometry>
@@ -219,25 +219,25 @@
       <material>Gazebo/DarkGrey</material>
     </gazebo> -->
-  <joint name="$(arg prefix)/navsat_joint" type="fixed">
-    <parent link="$(arg prefix)/chassis_link" />
-    <child link="$(arg prefix)/navsat_link" />
+  <joint name="$(arg prefix)_navsat_joint" type="fixed">
+    <parent link="$(arg prefix)_chassis_link" />
+    <child link="$(arg prefix)_navsat_link" />
     <origin xyz="-0.180 0.126 0.1815" />
   </joint>
-  <link name="$(arg prefix)/mid_mount"></link>
-  <joint name="$(arg prefix)/mid_mount_joint" type="fixed">
-    <parent link="$(arg prefix)/chassis_link" />
-    <child link="$(arg prefix)/mid_mount" />
+  <link name="$(arg prefix)_mid_mount"></link>
+  <joint name="$(arg prefix)_mid_mount_joint" type="fixed">
+    <parent link="$(arg prefix)_chassis_link" />
+    <child link="$(arg prefix)_mid_mount" />
     <origin xyz="0 0 ${chassis_height}" />
   </joint>
-  <link name="$(arg prefix)/rear_mount"></link>
-  <joint name="$(arg prefix)/rear_mount_joint" type="fixed">
-    <parent link="$(arg prefix)/mid_mount" />
-    <child link="$(arg prefix)/rear_mount" />
+  <link name="$(arg prefix)_rear_mount"></link>
+  <joint name="$(arg prefix)_rear_mount_joint" type="fixed">
+    <parent link="$(arg prefix)_mid_mount" />
+    <child link="$(arg prefix)_rear_mount" />
     <origin xyz="${-mount_spacing} 0 0" />
   </joint>
-  <link name="$(arg prefix)/front_mount"></link>
-  <joint name="$(arg prefix)/front_mount_joint" type="fixed">
-    <parent link="$(arg prefix)/mid_mount" />
-    <child link="$(arg prefix)/front_mount" />
+  <link name="$(arg prefix)_front_mount"></link>
+  <joint name="$(arg prefix)_front_mount_joint" type="fixed">
+    <parent link="$(arg prefix)_mid_mount" />
+    <child link="$(arg prefix)_front_mount" />
     <origin xyz="0 0 0" />
   </joint>
@@ -253,20 +253,20 @@
       </xacro:unless>
     </hardware>
-    <joint name="$(arg prefix)/front_left_wheel_joint">
-      <command_interface name="velocity"/>
-      <state_interface name="position"/>
-      <state_interface name="velocity"/>
-    </joint>
-    <joint name="$(arg prefix)/rear_left_wheel_joint">
-      <command_interface name="velocity"/>
-      <state_interface name="position"/>
-      <state_interface name="velocity"/>
-    </joint>
-    <joint name="$(arg prefix)/front_right_wheel_joint">
-      <command_interface name="velocity"/>
-      <state_interface name="position"/>
-      <state_interface name="velocity"/>
-    </joint>
-    <joint name="$(arg prefix)/rear_right_wheel_joint">
+    <joint name="$(arg prefix)_front_left_wheel_joint">
+      <command_interface name="velocity"/>
+      <state_interface name="position"/>
+      <state_interface name="velocity"/>
+    </joint>
+    <joint name="$(arg prefix)_rear_left_wheel_joint">
+      <command_interface name="velocity"/>
+      <state_interface name="position"/>
+      <state_interface name="velocity"/>
+    </joint>
+    <joint name="$(arg prefix)_front_right_wheel_joint">
+      <command_interface name="velocity"/>
+      <state_interface name="position"/>
+      <state_interface name="velocity"/>
+    </joint>
+    <joint name="$(arg prefix)_rear_right_wheel_joint">
       <command_interface name="velocity"/>
       <state_interface name="position"/>

Commit message: fix: namespacing for jackal and pallet_truck

File: jackal_description/urdf/accessories.urdf.xacro (robot description, xacro)
@@ -32,5 +32,5 @@
     <xacro:property name="tower" value="$(optenv JACKAL_LASER_TOWER 0)" />
     <xacro:property name="prefix" value="$(optenv JACKAL_LASER_PREFIX ${mount})" />
-    <xacro:property name="parent" value="$(optenv JACKAL_LASER_PARENT jackal_${mount}_mount)" />
+    <xacro:property name="parent" value="$(optenv JACKAL_LASER_PARENT ${namespace}/${mount}_mount)" />
     <xacro:property name="lidar_model" value="$(optenv JACKAL_LASER_MODEL ust10)" />
     <!-- SICK LMS1xx -->

File: jackal_description/urdf/jackal.urdf_underscores.xacro (robot description, xacro)
@@ -55,5 +55,5 @@
     </gazebo>
     <joint name="${wheel_prefix}_wheel_joint" type="continuous">
-      <parent link="$(arg prefix)/chassis_link"/>
+      <parent link="$(arg prefix)_chassis_link"/>
       <child link="${wheel_prefix}_wheel_link" />
       <xacro:insert_block name="joint_pose" />
@@ -72,23 +72,23 @@
     </transmission>
   </xacro:macro>
-  <xacro:wheel wheel_prefix="$(arg prefix)/front_left">
+  <xacro:wheel wheel_prefix="$(arg prefix)_front_left">
     <origin xyz="${wheelbase/2} ${track/2} ${wheel_vertical_offset}" rpy="0 0 0" />
   </xacro:wheel>
-  <xacro:wheel wheel_prefix="$(arg prefix)/front_right">
+  <xacro:wheel wheel_prefix="$(arg prefix)_front_right">
     <origin xyz="${wheelbase/2} ${-track/2} ${wheel_vertical_offset}" rpy="0 0 0" />
   </xacro:wheel>
-  <xacro:wheel wheel_prefix="$(arg prefix)/rear_left">
+  <xacro:wheel wheel_prefix="$(arg prefix)_rear_left">
     <origin xyz="${-wheelbase/2} ${track/2} ${wheel_vertical_offset}" rpy="0 0 0" />
   </xacro:wheel>
-  <xacro:wheel wheel_prefix="$(arg prefix)/rear_right">
+  <xacro:wheel wheel_prefix="$(arg prefix)_rear_right">
     <origin xyz="${-wheelbase/2} ${-track/2} ${wheel_vertical_offset}" rpy="0 0 0" />
   </xacro:wheel>
-  <link name="$(arg prefix)/base_link"></link>
-  <joint name="$(arg prefix)/base_link_joint" type="fixed">
+  <link name="$(arg prefix)_base_link"></link>
+  <joint name="$(arg prefix)_base_link_joint" type="fixed">
     <origin xyz="0 0 0" rpy="0 0 0" />
-    <parent link="$(arg prefix)/base_link"/>
-    <child link="$(arg prefix)/chassis_link" />
-  </joint>
-  <link name="$(arg prefix)/chassis_link">
+    <parent link="$(arg prefix)_base_link"/>
+    <child link="$(arg prefix)_chassis_link" />
+  </joint>
+  <link name="$(arg prefix)_chassis_link">
     <visual>
       <origin xyz="0 0 ${footprint_vertical_offset}" rpy="${PI/2} 0 ${PI/2}"/>
@@ -118,5 +118,5 @@
     </gazebo> -->
   <xacro:unless value="$(optenv JACKAL_FRONT_ACCESSORY_FENDER 0)">
-    <link name="$(arg prefix)/front_fender_link">
+    <link name="$(arg prefix)_front_fender_link">
       <visual>
         <geometry>
@@ -131,5 +131,5 @@
   </xacro:unless>
   <xacro:if value="$(optenv JACKAL_FRONT_ACCESSORY_FENDER 0)">
-    <link name="$(arg prefix)/front_fender_link">
+    <link name="$(arg prefix)_front_fender_link">
       <visual>
         <geometry>
@@ -142,18 +142,18 @@
       <material>Gazebo/Yellow</material>
     </gazebo> -->
-    <link name="$(arg prefix)/front_fender_accessory_link"/>
-    <joint name="$(arg prefix)/front_fender_accessory_joint" type="fixed">
+    <link name="$(arg prefix)_front_fender_accessory_link"/>
+    <joint name="$(arg prefix)_front_fender_accessory_joint" type="fixed">
       <origin xyz="0.25629 0 0.07455" rpy="${PI} 0 0" />
-      <parent link="$(arg prefix)/front_fender_link" />
-      <child link="$(arg prefix)/front_fender_accessory_link" />
+      <parent link="$(arg prefix)_front_fender_link" />
+      <child link="$(arg prefix)_front_fender_accessory_link" />
     </joint>
   </xacro:if>
-  <joint name="$(arg prefix)/front_fender_joint" type="fixed">
+  <joint name="$(arg prefix)_front_fender_joint" type="fixed">
     <origin xyz="0 0 0" rpy="0 0 0"/>
-    <parent link="$(arg prefix)/chassis_link" />
-    <child link="$(arg prefix)/front_fender_link" />
+    <parent link="$(arg prefix)_chassis_link" />
+    <child link="$(arg prefix)_front_fender_link" />
   </joint>
   <xacro:unless value="$(optenv JACKAL_REAR_ACCESSORY_FENDER 0)">
-    <link name="$(arg prefix)/rear_fender_link">
+    <link name="$(arg prefix)_rear_fender_link">
       <visual>
         <geometry>
@@ -168,5 +168,5 @@
   </xacro:unless>
   <xacro:if value="$(optenv JACKAL_REAR_ACCESSORY_FENDER 0)">
-    <link name="$(arg prefix)/rear_fender_link">
+    <link name="$(arg prefix)_rear_fender_link">
       <visual>
         <geometry>
@@ -179,15 +179,15 @@
       <material>Gazebo/Yellow</material>
     </gazebo> -->
-    <link name="$(arg prefix)/rear_fender_accessory_link"/>
-    <joint name="$(arg prefix)/rear_fender_accessory_joint" type="fixed">
+    <link name="$(arg prefix)_rear_fender_accessory_link"/>
+    <joint name="$(arg prefix)_rear_fender_accessory_joint" type="fixed">
       <origin xyz="0.25629 0 0.07455" rpy="${PI} 0 0" />
-      <parent link="$(arg prefix)/rear_fender_link" />
-      <child link="$(arg prefix)/rear_fender_accessory_link" />
+      <parent link="$(arg prefix)_rear_fender_link" />
+      <child link="$(arg prefix)_rear_fender_accessory_link" />
     </joint>
   </xacro:if>
-  <joint name="$(arg prefix)/rear_fender_joint" type="fixed">
+  <joint name="$(arg prefix)_rear_fender_joint" type="fixed">
     <origin xyz="0 0 0" rpy="0 0 ${PI}"/>
-    <parent link="$(arg prefix)/chassis_link" />
-    <child link="$(arg prefix)/rear_fender_link" />
+    <parent link="$(arg prefix)_chassis_link" />
+    <child link="$(arg prefix)_rear_fender_link" />
   </joint>
   <!-- TODO Make this internal_imu_link or something, and use a mixed-in xacro
@@ -195,5 +195,5 @@
        always points to the "active" IMU. When an upgrade IMU is connected, the
        internal_imu_link should remain, but imu_link should point to the upgrade one. -->
-  <link name="$(arg prefix)/imu_link">
+  <link name="$(arg prefix)_imu_link">
     <inertial>
       <mass value="0.001"/>
@@ -202,10 +202,10 @@
     </inertial>
   </link>
-  <joint name="$(arg prefix)/imu_joint" type="fixed">
-    <parent link="$(arg prefix)/chassis_link" />
-    <child link="$(arg prefix)/imu_link" />
+  <joint name="$(arg prefix)_imu_joint" type="fixed">
+    <parent link="$(arg prefix)_chassis_link" />
+    <child link="$(arg prefix)_imu_link" />
   </joint>
   <!-- TODO Same note as applies to imu_link -->
-  <link name="$(arg prefix)/navsat_link">
+  <link name="$(arg prefix)_navsat_link">
     <visual>
       <geometry>
@@ -219,25 +219,25 @@
       <material>Gazebo/DarkGrey</material>
     </gazebo> -->
-  <joint name="$(arg prefix)/navsat_joint" type="fixed">
-    <parent link="$(arg prefix)/chassis_link" />
-    <child link="$(arg prefix)/navsat_link" />
+  <joint name="$(arg prefix)_navsat_joint" type="fixed">
+    <parent link="$(arg prefix)_chassis_link" />
+    <child link="$(arg prefix)_navsat_link" />
     <origin xyz="-0.180 0.126 0.1815" />
   </joint>
-  <link name="$(arg prefix)/mid_mount"></link>
-  <joint name="$(arg prefix)/mid_mount_joint" type="fixed">
-    <parent link="$(arg prefix)/chassis_link" />
-    <child link="$(arg prefix)/mid_mount" />
+  <link name="$(arg prefix)_mid_mount"></link>
+  <joint name="$(arg prefix)_mid_mount_joint" type="fixed">
+    <parent link="$(arg prefix)_chassis_link" />
+    <child link="$(arg prefix)_mid_mount" />
     <origin xyz="0 0 ${chassis_height}" />
   </joint>
-  <link name="$(arg prefix)/rear_mount"></link>
-  <joint name="$(arg prefix)/rear_mount_joint" type="fixed">
-    <parent link="$(arg prefix)/mid_mount" />
-    <child link="$(arg prefix)/rear_mount" />
+  <link name="$(arg prefix)_rear_mount"></link>
+  <joint name="$(arg prefix)_rear_mount_joint" type="fixed">
+    <parent link="$(arg prefix)_mid_mount" />
+    <child link="$(arg prefix)_rear_mount" />
     <origin xyz="${-mount_spacing} 0 0" />
   </joint>
-  <link name="$(arg prefix)/front_mount"></link>
-  <joint name="$(arg prefix)/front_mount_joint" type="fixed">
-    <parent link="$(arg prefix)/mid_mount" />
-    <child link="$(arg prefix)/front_mount" />
+  <link name="$(arg prefix)_front_mount"></link>
+  <joint name="$(arg prefix)_front_mount_joint" type="fixed">
+    <parent link="$(arg prefix)_mid_mount" />
+    <child link="$(arg prefix)_front_mount" />
     <origin xyz="0 0 0" />
   </joint>
@@ -253,20 +253,20 @@
       </xacro:unless>
     </hardware>
-    <joint name="$(arg prefix)/front_left_wheel_joint">
-      <command_interface name="velocity"/>
-      <state_interface name="position"/>
-      <state_interface name="velocity"/>
-    </joint>
-    <joint name="$(arg prefix)/rear_left_wheel_joint">
-      <command_interface name="velocity"/>
-      <state_interface name="position"/>
-      <state_interface name="velocity"/>
-    </joint>
-    <joint name="$(arg prefix)/front_right_wheel_joint">
-      <command_interface name="velocity"/>
-      <state_interface name="position"/>
-      <state_interface name="velocity"/>
-    </joint>
-    <joint name="$(arg prefix)/rear_right_wheel_joint">
+    <joint name="$(arg prefix)_front_left_wheel_joint">
+      <command_interface name="velocity"/>
+      <state_interface name="position"/>
+      <state_interface name="velocity"/>
+    </joint>
+    <joint name="$(arg prefix)_rear_left_wheel_joint">
+      <command_interface name="velocity"/>
+      <state_interface name="position"/>
+      <state_interface name="velocity"/>
+    </joint>
+    <joint name="$(arg prefix)_front_right_wheel_joint">
+      <command_interface name="velocity"/>
+      <state_interface name="position"/>
+      <state_interface name="velocity"/>
+    </joint>
+    <joint name="$(arg prefix)_rear_right_wheel_joint">
       <command_interface name="velocity"/>
       <state_interface name="position"/>
