Commit message: Update sensor plugins to jazzy version. Fix control.yaml.

File: jackal_description/urdf/jackal.urdf.xacro (robot description, xacro)
@@ -49,7 +49,7 @@
       <selfCollide>false</selfCollide>
       <mu1 value="0.5"/>
-      <mu2 value="0.5"/>
+      <mu2 value="0.1"/>
       <kp value="10000000.0" />
-      <kd value="1" />
+      <kd value="10" />
       <fdir1 value="1 0 0"/>
     </gazebo>
@@ -59,4 +59,6 @@
       <xacro:insert_block name="joint_pose" />
       <axis xyz="0 1 0" />
+      <limit effort="8.0" velocity="4.0"/>
+      <dynamics damping="0.0" friction="0.0"/>
     </joint>
     <!-- In reality, Jackal has only two motors, one per side. However, it's more
@@ -244,5 +246,5 @@
   <!-- ROS2 controls -->
   <ros2_control name="jackal_hardware" type="system">
-      <hardware>
+    <hardware>
       <xacro:if value="$(arg is_sim)">
         <plugin>gz_ros2_control/GazeboSimSystem</plugin>

Commit message: Max speed capping fixed. It was a limit on the joint. Cleaned up code.

File: jackal_description/urdf/jackal.urdf.xacro (robot description, xacro)
@@ -49,5 +49,5 @@
       <selfCollide>false</selfCollide>
       <mu1 value="0.5"/>
-      <mu2 value="0.1"/>
+      <mu2 value="0.5"/>
       <kp value="10000000.0" />
       <kd value="10" />
@@ -59,6 +59,4 @@
       <xacro:insert_block name="joint_pose" />
       <axis xyz="0 1 0" />
-      <limit effort="8.0" velocity="4.0"/>
-      <dynamics damping="0.0" friction="0.0"/>
     </joint>
     <!-- In reality, Jackal has only two motors, one per side. However, it's more
